File: microcntr.kicad_sch (KiCad schematic)
At the start: 165 parts, among them IC1 M24512-RDW6TP, IC2 ADF4156BRUZ, IC3 ADM7160AUJZ-3.3-R7, IC4 ADM7160AUJZ-3.3-R7, J1 U.FL, J10 U.FL, J4 Conn_01x16, J5 RF2-04A-T-00-50-G, J6 Conn_01x12, J7 USB_B_Micro, J8 RF2-04A-T-00-50-G, J9 RF2-04A-T-00-50-G, Q1 BSH105,215, Q2 BC69PASX, Q3 BCV62C, Q4 BFU550WF, U1 SN74LVC1G80QDCKRQ1, U11 SN74LVC1G97DCKR, U12 TLV3601DCKR, U14 MAX-M10S-00B, U15 TLV3601DCKR, U16 LMT85DCKR, U17 TLV9162IDDFR, U18 SN74LVC1G80QDCKRQ1, U2 ADR381ARTZ-R2, U3 TLV3601DCKR, U4 TLV9162IDDFR, U5 SN74LVC1G80QDCKRQ1, U6 SN74LVC1G97DCKR, U7 STM32F410RBT6, U8 SN74LVC1G97DCKR, U9 FT230XS, Y2 CCHD-575-50-100.000

Commit message: added buglist
Other:
- note added: "Aliexpress SMA-SMA SMA-F - U.FL CONSMA020.062-G equivalent Scope probe? Nadelfeile Lötkolben Uhrmacherlupe x10+ GPS Ant"
- note removed: "Aliexpress SMA-SMA SMA-F - U.FL CONSMA020.062-G equivalent Scope probe? Nadelfeile Lötkolben Uhrmacherlupe x10+"
Changed lines of the file:
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@@
     (effects (font (size 1.27 1.27)) (justify left bottom))
   )
-  (text "Aliexpress\nSMA-SMA\nSMA-F - U.FL\nCONSMA020.062-G equivalent\nScope probe?\nNadelfeile\nLötkolben\nUhrmacherlupe x10+"
+  (text "Aliexpress\nSMA-SMA\nSMA-F - U.FL\nCONSMA020.062-G equivalent\nScope probe?\nNadelfeile\nLötkolben\nUhrmacherlupe x10+\nGPS Ant"
     (at 15.24 124.46 0)
     (effects (font (size 2.54 2.54)) (justify left bottom))

Commit message: buglist new bugs
Other:
- note added: "<10 MHz"
- note added: ">=10 MHz"
- note added: "good setting: 2k"
Changed lines of the file:
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@@
     (effects (font (size 1.27 1.27)) (justify left bottom))
   )
+  (text "good setting: 2k" (at 341.63 350.52 0)
+    (effects (font (size 1.27 1.27)) (justify left bottom))
+  )
   (text "DUT IN Low" (at 32.385 181.61 0)
     (effects (font (size 3 3)) (justify left bottom))
   )
+  (text ">=10 MHz" (at 142.24 208.915 0)
+    (effects (font (size 1.5 1.5)) (justify left bottom))
+  )
   (text "FMPI2C1_SDA" (at 429.895 102.87 0)
     (effects (font (size 1.27 1.27)) (justify left bottom))
@@
     (effects (font (size 1.27 1.27)) (justify right bottom))
   )
+  (text "<10 MHz" (at 143.51 225.425 0)
+    (effects (font (size 1.5 1.5)) (justify left bottom))
+  )
   (text "15mA" (at 122.555 335.28 0)
     (effects (font (size 1.27 1.27) (thickness 0.254) bold) (justify left bottom))
@@
       (effects (font (size 1.27 1.27)) (justify left))
     )
-    (property "Value" "51R" (id 1) (at 144.78 207.01 90)
+    (property "Value" "51R" (id 1) (at 141.605 207.01 90)
       (effects (font (size 1.27 1.27)) (justify left))
     )
@@
       (effects (font (size 1.27 1.27)) hide)
     )
-    (property "Data" "10k 0.1W" (id 4) (at 351.79 356.87 0))
+    (property "Data" "10k 0.1W" (id 4) (at 351.79 356.87 0)
+      (effects (font (size 1.27 1.27)) hide)
+    )
     (property "Manufacturer_Part_Number" "3214J-2-103E" (id 5) (at 359.41 354.33 0)
       (effects (font (size 1.27 1.27)) hide)

Commit message: added comments
Other:
- note added: "SEL 0 -> IN1 TIMEPULSE_HSI"
- note added: "SEL 0 -> IN1 int ref"
- note added: "SEL 1 -> IN0 CAL_100M"
- note added: "SEL 1 -> IN0 ext ref"
- note removed: "SEL 0 -> IN1"
- note removed: "SEL 1 -> IN0"
Changed lines of the file:
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@@
     (effects (font (size 1.27 1.27)) (justify left bottom))
   )
-  (text "SEL 0 -> IN1" (at 200.66 294.005 0)
+  (text "SEL 0 -> IN1 int ref" (at 200.66 294.005 0)
     (effects (font (size 2.54 2.54)) (justify left bottom))
   )
@@
     (effects (font (size 3 3) (thickness 0.6) bold) (justify right bottom))
   )
+  (text "SEL 1 -> IN0 CAL_100M\n" (at 116.84 243.205 0)
+    (effects (font (size 2.54 2.54)) (justify left bottom))
+  )
   (text "Disabled at startup!" (at 83.82 294.005 0)
     (effects (font (size 2.54 2.54)) (justify left bottom))
@@
     (effects (font (size 1.27 1.27)) (justify left bottom))
   )
-  (text "SEL 1 -> IN0\n" (at 200.66 289.56 0)
+  (text "SEL 1 -> IN0 ext ref\n" (at 200.66 289.56 0)
     (effects (font (size 2.54 2.54)) (justify left bottom))
   )
@@
     (effects (font (size 1.27 1.27)) (justify left bottom))
   )
+  (text "SEL 0 -> IN1 TIMEPULSE_HSI" (at 116.84 247.65 0)
+    (effects (font (size 2.54 2.54)) (justify left bottom))
+  )
   (text "current limit 0.22A 1W" (at 431.165 354.33 0)

Commit message: new buglist entries
Other:
- note added: "BUG: TLV3603 LE# should be floating or have pulldown"
- note added: "TIM6: display delays TIM11: chibios TIM1: timepulse measure"
Changed lines of the file:
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@@
     (effects (font (size 4 4) (thickness 0.8) bold) (justify left bottom))
+  )
+  (text "BUG: TLV3603 LE# should be floating or have pulldown"
+    (at 97.79 281.305 0)
+    (effects (font (size 2 2) (thickness 0.4) bold) (justify left bottom))
   )
   (text "0°   1.567V\n100° 0.737V\npush-pull +/- 50uA\n" (at 313.69 373.38 0)
@@
     (effects (font (size 2.54 2.54)) (justify left bottom))
   )
+  (text "BUG: TLV3603 LE# should be floating or have pulldown"
+    (at 85.725 215.9 0)
+    (effects (font (size 2 2) (thickness 0.4) bold) (justify left bottom))
+  )
   (text "TIM5_CH3" (at 430.53 113.03 0)
     (effects (font (size 1.27 1.27)) (justify left bottom))
@@
   (text "20mA?" (at 464.185 28.575 0)
     (effects (font (size 1.27 1.27) (thickness 0.254) bold) (justify left bottom))
+  )
+  (text "TIM6: display delays\nTIM11: chibios\nTIM1: timepulse measure"
+    (at 278.765 109.22 0)
+    (effects (font (size 3 3)) (justify left bottom))
   )
   (text "Common mode\nChoke" (at 85.725 46.355 0)
@@
     (effects (font (size 1.27 1.27)) (justify left bottom))
   )
+  (text "BUG: TLV3603 LE# should be floating or have pulldown"
+    (at 314.96 259.08 0)
+    (effects (font (size 2 2) (thickness 0.4) bold) (justify left bottom))
+  )
   (text "TODO CONSMA020.062-G" (at 15.24 139.065 0)

Commit message: filled in buglist
Other:
- note added: "~{pulse} rising TIM5_CH1 Capture -> DMA -> TIM5 TRGO -> ADC CH10 injected conv TIM9 TI2 triggered one pulse on OC1 -> discharge pulse (connecting to U5.4 enables samplig the offset. necessary to compensate sub-threshold leakage of diodes)"
- note removed: "~{pulse} rising TIM5_CH1 Capture -> DMA -> TIM5 TRGO -> ADC CH10 injected conv TIM9 TI2 triggered one pulse on OC1 -> discharge pulse"
Changed lines of the file:
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@@
     (effects (font (size 1.27 1.27) (thickness 0.254) bold) (justify left bottom))
   )
-  (text "~{pulse} rising\nTIM5_CH1 Capture \n	-> DMA\n  	-> TIM5 TRGO\n		-> ADC CH10 injected conv\nTIM9 TI2 triggered one pulse on OC1\n	-> discharge pulse"
-    (at 187.96 135.255 0)
+  (text "~{pulse} rising\nTIM5_CH1 Capture \n	-> DMA\n  	-> TIM5 TRGO\n		-> ADC CH10 injected conv\nTIM9 TI2 triggered one pulse on OC1\n	-> discharge pulse\n(connecting to U5.4 enables samplig the \noffset. necessary to compensate sub-threshold\nleakage of diodes)"
+    (at 187.325 148.59 0)
     (effects (font (size 3 3)) (justify left bottom))
   )
