File: microcntr.kicad_sch (KiCad schematic)
At the start: 165 parts, among them IC1 M24512-RDW6TP, IC2 ADF4156BRUZ, IC3 ADM7160AUJZ-3.3-R7, IC4 ADM7160AUJZ-3.3-R7, J1 U.FL, J10 U.FL, J4 Conn_01x16, J5 RF2-04A-T-00-50-G, J6 Conn_01x12, J7 USB_B_Micro, J8 RF2-04A-T-00-50-G, J9 RF2-04A-T-00-50-G, Q1 BSH105,215, Q2 BC69PASX, Q3 BCV62C, Q4 BFU550WF, U1 SN74LVC1G80QDCKRQ1, U11 SN74LVC1G97DCKR, U12 TLV3601DCKR, U14 MAX-M10S-00B, U15 TLV3601DCKR, U16 LMT85DCKR, U17 TLV9162IDDFR, U18 SN74LVC1G80QDCKRQ1, U2 ADR381ARTZ-R2, U3 TLV3601DCKR, U4 TLV9162IDDFR, U5 SN74LVC1G80QDCKRQ1, U6 SN74LVC1G97DCKR, U7 STM32F410RBT6, U8 SN74LVC1G97DCKR, U9 FT230XS, Y2 CCHD-575-50-100.000

Commit message: added comment
Other:
- note added: "TIM6: display delays TIM11: chibios TIM1: timepulse measure (start as slave of TIM5)"
- note removed: "TIM6: display delays TIM11: chibios TIM1: timepulse measure"
Changed lines of the file:
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@@
     (effects (font (size 1.27 1.27) (thickness 0.254) bold) (justify left bottom))
   )
-  (text "TIM6: display delays\nTIM11: chibios\nTIM1: timepulse measure"
-    (at 278.765 109.22 0)
+  (text "TIM6: display delays\nTIM11: chibios\nTIM1: timepulse measure (start as slave of TIM5)"
+    (at 246.38 108.585 0)
     (effects (font (size 3 3)) (justify left bottom))
   )

Commit message: some comments
Other:
- note added: "<3ppm 1st year, <1ppm thereafter"
- note added: "Pullup on button B"
- note added: "good setting: 3.3k. (almost no overshoot)"
- note added: "~{pulse} rising TIM5_CH1 Capture -> DMA (probably not useful: handling of timer overflows?) -> TIM5 TRGO -> ADC CH10 injected conv (no DMA possible) TIM9 TI2 triggered one pulse on OC1 -> discharge pulse (connecting to U5.4 enables samplig the offset. necessary to compensate sub-threshold leakage of diodes) Just trigger adc isr and collect tim capture and ADC value"
- note added: "±50ppm 0°C ~ 70°C"
- note removed: "good setting: 2k"
- note removed: "~{pulse} rising TIM5_CH1 Capture -> DMA -> TIM5 TRGO -> ADC CH10 injected conv TIM9 TI2 triggered one pulse on OC1 -> discharge pulse (connecting to U5.4 enables samplig the offset. necessary to compensate sub-threshold leakage of diodes)"
Changed lines of the file:
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@@
     (effects (font (size 1.27 1.27)) (justify left bottom))
+  )
+  (text "Pullup on button B" (at 565.15 62.23 180)
+    (effects (font (size 1 1)) (justify right bottom))
   )
   (text "TLV3601 has no pin5 LE/HYS\n" (at 97.79 278.13 0)
@@
     (effects (font (size 4 4) (thickness 0.8) bold) (justify left bottom))
   )
+  (text "<3ppm 1st year, <1ppm thereafter" (at 154.305 316.23 0)
+    (effects (font (size 1.27 1.27)) (justify left bottom))
+  )
   (text "BUG: TLV3603 LE# should be floating or have pulldown"
     (at 97.79 281.305 0)
@@
     (effects (font (size 1.27 1.27)) (justify left bottom))
   )
-  (text "good setting: 2k" (at 341.63 350.52 0)
+  (text "good setting: 3.3k. \n(almost no overshoot)" (at 341.63 350.52 0)
     (effects (font (size 1.27 1.27)) (justify left bottom))
   )
@@
   )
   (text "TIM6: display delays\nTIM11: chibios\nTIM1: timepulse measure (start as slave of TIM5)"
-    (at 246.38 108.585 0)
-    (effects (font (size 3 3)) (justify left bottom))
+    (at 186.055 105.41 0)
+    (effects (font (size 2 2)) (justify left bottom))
+  )
+  (text "±50ppm 0°C ~ 70°C" (at 154.305 313.69 0)
+    (effects (font (size 1.27 1.27)) (justify left bottom))
   )
   (text "Common mode\nChoke" (at 85.725 46.355 0)
@@
     (effects (font (size 1.27 1.27) (thickness 0.254) bold) (justify left bottom))
   )
-  (text "~{pulse} rising\nTIM5_CH1 Capture \n	-> DMA\n  	-> TIM5 TRGO\n		-> ADC CH10 injected conv\nTIM9 TI2 triggered one pulse on OC1\n	-> discharge pulse\n(connecting to U5.4 enables samplig the \noffset. necessary to compensate sub-threshold\nleakage of diodes)"
-    (at 187.325 148.59 0)
-    (effects (font (size 3 3)) (justify left bottom))
+  (text "~{pulse} rising\nTIM5_CH1 Capture \n	-> DMA (probably not useful: handling of timer overflows?)\n  	-> TIM5 TRGO\n		-> ADC CH10 injected conv (no DMA possible)\nTIM9 TI2 triggered one pulse on OC1\n	-> discharge pulse\n(connecting to U5.4 enables samplig the \noffset. necessary to compensate sub-threshold\nleakage of diodes)\n\nJust trigger adc isr and collect tim capture and ADC value"
+    (at 185.42 158.115 0)
+    (effects (font (size 2 2)) (justify left bottom))
   )
   (text "67° 1.02V" (at 337.82 370.84 0)
